File: esp8266_ir_transmitter/schematics/esp8266_ir_transmitter.kicad_pcb (KiCad board)
At the start: 2 copper layers, 30 x 52 mm, 34 parts, among them P1 SERIAL, P10 TEMP1, P11 GND, P12 AUX, P13 GND, P14 3.3V, P15 AC unit 5V, P2 IR LED, P3 5V, P4 3V3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

Commit message: PCB revision 1
Parts:
- added C6: 100n, Capacitors_SMD:C_0805_HandSoldering, F.Cu at (52.1, 58.4)
- added C7: 100n, Capacitors_SMD:C_0805_HandSoldering, F.Cu at (52.1, 63.5)
- added D3: LED, LEDs:LED_0805_HandSoldering, F.Cu at (48.9, 40.1)
- added R12: 1k, Resistors_SMD:R_0805_HandSoldering, F.Cu at (50.9, 36.2)
- P10: value TEMP1 -> T1
- P7: value TEMP0 -> T0
- moved Q1 1.59 mm to (52.4, 40.4)
- moved P7 1.27 mm to (49.5, 55.2)
Routing:
- net Net-(D3-Pad1): track 6.88 -> 12.2 mm
- net GND: track 43.6 -> 47.0 mm, vias 8 -> 9
- net +3V3: track 32.2 -> 35.3 mm, vias 5 -> 6
- net Net-(D3-Pad2): track 0.00 -> 2.80 mm
- net Net-(C7-Pad1): track 10.1 -> 11.6 mm
- net Net-(C6-Pad1): track 15.0 -> 16.1 mm
- net /GPIO14: track 28.4 -> 27.7 mm
